File: EclectronicsProject2.sch (KiCad schematic (older format))
At the start: 87 parts, among them J2 Conn_01x08, J3 Conn_01x10, J4 Conn_01x06, J6 Conn_01x08, J7 PowerJack3P, Q1 Q_PMOS_DGS, Q2B Q_NMOS_DGS, Q5 Q_PMOS_DGS, U11 TPS62290DRVR, U1A FE310-G000, U2 TXS0108E, U3 TXS0108E, U4 TXS0104E, U5 IS25LP0128, U7 TPS62133RGTT, U8 TPS62290DRVR, Y1 clock

Commit message: design rules check complete
Parts:
- U98: renamed from U?; Part (none) -> BM71BLES1FC2-0002AA-ND
- gave numbers to parts that had none: 6
- renumbered Q2B to Q21, U1A to U19
Connections:
- net GND: now also U2.11 (GND)
- net HCI_RXD: now also J4.2 (Pin_2)
- net HCI_TXD: now also J4.1 (Pin_1)
- net P0_2/LED: now also J4.6 (Pin_6)
- net TP1 renamed VDD_1V8
- net VDD_3V3_MOFF renamed IVDD

Commit message: final part number
Parts:
- U5: Part (none) -> IS25LP128-JBLE
- clk1: Part (none) -> SIT1533AC-H5-D14-
Changed lines of the file:
@@
 F 2 "" H 9375 8725 60  0001 C CNN
 F 3 "" H 9375 8725 60  0001 C CNN
+F 4 "IS25LP128-JBLE" H 9375 8725 60  0001 C CNN "Part"
 	1    9375 8725
 	1    0    0    -1
@@
 F 2 "" H 1725 8800 39  0001 C CNN
 F 3 "" H 1725 8800 39  0001 C CNN
+F 4 "SIT1533AC-H5-D14-" H 1725 8800 60  0001 C CNN "Part"
 	1    1725 8800
 	1    0    0    -1

Commit message: arduino time
Parts:
- C1, C10, C11, C12, C13, C16, C17, C18, C19, C2, C20, C21, C22, C23, C3, C4, C42, C44, C45, C48, C49, C5, C51, C54, C6, C8, C9, C99: footprint (none) -> Capacitors_SMD:C_0603
- C43, C46, C47, C50, C52, C55, C98: footprint (none) -> Capacitors_SMD:C_0805
- D1, D4: footprint (none) -> project2:BAT54-SC-59
- D10, D9: footprint (none) -> LEDs:LED_0805
- D13: footprint (none) -> project2:DB2W40300LCT-ND
- D2, D5: footprint (none) -> project2:PBG1010603
- J1, J2, J6: footprint (none) -> Pin_Headers:Pin_Header_Straight_1x08_Pitch1.00mm
- J3: footprint (none) -> Pin_Headers:Pin_Header_Straight_1x10_Pitch1.00mm
- J4: footprint (none) -> Pin_Headers:Pin_Header_Straight_1x06_Pitch1.00mm
- J7: footprint (none) -> Connectors:BARREL_JACK
- L1, L2, L3: footprint (none) -> project2:490-10649-1-ND
- Q1, Q5: footprint (none) -> TO_SOT_Packages_SMD:SOT-23
- Q21: footprint (none) -> TO_SOT_Packages_SMD:SOT-363_SC-70-6
- R1, R13, R2, R27, R28, R3, R30, R31, R34, R35, R36, R37, R39, R5, R6, R9, R97: footprint (none) -> Resistors_SMD:R_0603
- S1, S2: footprint (none) -> Buttons_Switches_SMD:SW_SPST_B3S-1000
- U11, U8: footprint (none) -> project2:296-27030-1-ND
- U2, U3: footprint (none) -> project2:296-24806-1-ND
- U4: footprint (none) -> Housings_DFN_QFN:Texas_S-PVQFN-N14_ThermalVias
- U5: footprint (none) -> Housings_SOIC:SOIJ-8_5.3x5.3mm_Pitch1.27mm
- U7: footprint (none) -> project2:296-30225-1-ND
- Y1: footprint (none) -> project2:TM16
- Y3: renamed from clk1; footprint (none) -> project2:SiT1533
- d12: footprint (none) -> project2:F5747CT-ND
