File: USBtoUART.sch (KiCad schematic (older format))
At the start: 30 parts

Commit message: updated values and part numbers
Parts:
- removed Q?: Q_PMOS_DGS, symbol Q_PMOS_DGS
- added Q3A: Q_NMOS_DGS, symbol Q_NMOS_DGS
- J5: renamed from J?; Part (none) -> A108263CTND
- U6: renamed from U?; Part (none) -> 768-1030-ND
- gave numbers to parts that had none: 27
Connections:
- net FT_RESET: now also Q3A.3 (S)
- net VDD_1V8: now also Q3A.2 (G)
- net at R23.2, U6.14 (RESET#): now also Q3A.1 (D)
- no-connect marks 3 -> 4
Other:
- note added: "USB to UART\n"
- moved on the sheet: C24, C25, C26, C27, C28, C29, C30, C31, C32, C33, C34, C35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

Commit message: design rules check complete
Parts:
- renumbered Q3A to Q31
Connections:
- net VPHY_FT: no longer names the net of C32.1, C33.1, FB2.1, U6.4 (VPHY)
- net VPLL_FT: no longer names the net of C24.1, C25.1, FB1.1, U6.9 (VPLL)
- no-connect marks 4 -> 31
Changed lines of the file:
@@
 $EndComp
 $Comp
-L GND #PWR?
+L GND #PWR051
 U 1 1 59CD8A85
 P 5875 6125
-F 0 "#PWR?" H 5875 5875 50  0001 C CNN
+F 0 "#PWR051" H 5875 5875 50  0001 C CNN
 F 1 "GND" H 5875 5975 50  0000 C CNN
 F 2 "" H 5875 6125 50  0001 C CNN
@@
 $EndComp
 $Comp
-L GND #PWR?
+L GND #PWR052
 U 1 1 59CD8AF0
 P 5100 5725
-F 0 "#PWR?" H 5100 5475 50  0001 C CNN
+F 0 "#PWR052" H 5100 5475 50  0001 C CNN
 F 1 "GND" H 5100 5575 50  0000 C CNN
 F 2 "" H 5100 5725 50  0001 C CNN
@@
 $EndComp
 $Comp
-L GND #PWR?
+L GND #PWR053
 U 1 1 59CD8FB6
 P 4900 5275
-F 0 "#PWR?" H 4900 5025 50  0001 C CNN
+F 0 "#PWR053" H 4900 5025 50  0001 C CNN
 F 1 "GND" H 4900 5125 50  0000 C CNN
 F 2 "" H 4900 5275 50  0001 C CNN
@@
 $EndComp
 $Comp
-L GND #PWR?
+L GND #PWR054
 U 1 1 59CD8FE5
 P 4150 5275
-F 0 "#PWR?" H 4150 5025 50  0001 C CNN
+F 0 "#PWR054" H 4150 5025 50  0001 C CNN
 F 1 "GND" H 4150 5125 50  0000 C CNN
 F 2 "" H 4150 5275 50  0001 C CNN
@@
 $EndComp
 $Comp
-L GND #PWR?
+L GND #PWR055
 U 1 1 59CD9A61
 P 5250 2675
-F 0 "#PWR?" H 5250 2425 50  0001 C CNN
+F 0 "#PWR055" H 5250 2425 50  0001 C CNN
 F 1 "GND" H 5250 2525 50  0000 C CNN
 F 2 "" H 5250 2675 50  0001 C CNN
@@
 $EndComp
 $Comp
-L GND #PWR?
+L GND #PWR056
 U 1 1 59CD9A84
 P 5250 2050
-F 0 "#PWR?" H 5250 1800 50  0001 C CNN
+F 0 "#PWR056" H 5250 1800 50  0001 C CNN
 F 1 "GND" H 5250 1900 50  0000 C CNN
 F 2 "" H 5250 2050 50  0001 C CNN
@@
 Wire Wire Line
 	6075 2475 6075 2650
-Text GLabel 5400 1475 0    60   Input ~ 0
-VPLL_FT
-Text GLabel 5400 2150 2    60   Input ~ 0
-VPHY_FT
-Wire Wire Line
-	5400 2150 5375 2150
-Wire Wire Line
-	5375 2150 5375 2225
-Wire Wire Line
-	5375 2225 5425 2225
-Wire Wire Line
-	5425 2225 5425 2275
-Wire Wire Line
-	5400 1475 5425 1475
-Wire Wire Line
-	5425 1475 5425 1650
 $Comp
 L C C34
@@
 Connection ~ 4075 2275
 $Comp
-L GND #PWR?
+L GND #PWR057
 U 1 1 59CDA7F6
 P 4075 3675
-F 0 "#PWR?" H 4075 3425 50  0001 C CNN
+F 0 "#PWR057" H 4075 3425 50  0001 C CNN
 F 1 "GND" H 4075 3525 50  0000 C CNN
 F 2 "" H 4075 3675 50  0001 C CNN
@@
 Connection ~ 4075 3225
 $Comp
-L GND #PWR?
+L GND #PWR058
 U 1 1 59CDAC6E
 P 5025 3650
-F 0 "#PWR?" H 5025 3400 50  0001 C CNN
+F 0 "#PWR058" H 5025 3400 50  0001 C CNN
 F 1 "GND" H 5025 3500 50  0000 C CNN
 F 2 "" H 5025 3650 50  0001 C CNN
@@
 $EndComp
 $Comp
-L GND #PWR?
+L GND #PWR059
 U 1 1 59CDB20A
 P 1525 4975
-F 0 "#PWR?" H 1525 4725 50  0001 C CNN
+F 0 "#PWR059" H 1525 4725 50  0001 C CNN
 F 1 "GND" H 1525 4825 50  0000 C CNN
 F 2 "" H 1525 4975 50  0001 C CNN
@@
 	2950 3850 2800 3850
 $Comp
-L GND #PWR?
+L GND #PWR060
 U 1 1 59CDB7AD
 P 3300 3400
-F 0 "#PWR?" H 3300 3150 50  0001 C CNN
+F 0 "#PWR060" H 3300 3150 50  0001 C CNN
 F 1 "GND" H 3300 3250 50  0000 C CNN
 F 2 "" H 3300 3400 50  0001 C CNN
@@
 Connection ~ 3225 4950
 $Comp
-L GND #PWR?
+L GND #PWR061
 U 1 1 59CDBD67
 P 5250 4675
-F 0 "#PWR?" H 5250 4425 50  0001 C CNN
+F 0 "#PWR061" H 5250 4425 50  0001 C CNN
 F 1 "GND" H 5250 4525 50  0000 C CNN
 F 2 "" H 5250 4675 50  0001 C CNN
@@
 $EndComp
 $Comp
-L GND #PWR?
+L GND #PWR062
 U 1 1 59CDD413
 P 7125 3725
-F 0 "#PWR?" H 7125 3475 50  0001 C CNN
+F 0 "#PWR062" H 7125 3475 50  0001 C CNN
 F 1 "GND" H 7125 3575 50  0000 C CNN
 F 2 "" H 7125 3725 50  0001 C CNN
@@
 $EndComp
 $Comp
-L GND #PWR?
+L GND #PWR063
 U 1 1 59CDD4A2
 P 7300 3725
-F 0 "#PWR?" H 7300 3475 50  0001 C CNN
+F 0 "#PWR063" H 7300 3475 50  0001 C CNN
 F 1 "GND" H 7300 3575 50  0000 C CNN
 F 2 "" H 7300 3725 50  0001 C CNN
@@
 $EndComp
 $Comp
-L GND #PWR?
+L GND #PWR064
 U 1 1 59CDDB0A
 P 7275 4625
-F 0 "#PWR?" H 7275 4375 50  0001 C CNN
+F 0 "#PWR064" H 7275 4375 50  0001 C CNN
 F 1 "GND" H 7275 4475 50  0000 C CNN
 F 2 "" H 7275 4625 50  0001 C CNN
@@
 Connection ~ 8250 2400
 $Comp
-L GND #PWR?
+L GND #PWR065
 U 1 1 59CDE9C3
 P 8525 2475
-F 0 "#PWR?" H 8525 2225 50  0001 C CNN
+F 0 "#PWR065" H 8525 2225 50  0001 C CNN
 F 1 "GND" H 8525 2325 50  0000 C CNN
 F 2 "" H 8525 2475 50  0001 C CNN
@@
 	8525 2400 8525 2475
 $Comp
-L GND #PWR?
+L GND #PWR066
 U 1 1 59CDEC87
 P 7425 2475
-F 0 "#PWR?" H 7425 2225 50  0001 C CNN
+F 0 "#PWR066" H 7425 2225 50  0001 C CNN
 F 1 "GND" H 7425 2325 50  0000 C CNN
 F 2 "" H 7425 2475 50  0001 C CNN
@@
 NoConn ~ 2800 4450
 $Comp
-L Q_NMOS_DGS Q3A
+L Q_NMOS_DGS Q31
 U 1 1 59DA777E
 P 2375 5650
-F 0 "Q3A" H 2575 5700 50  0000 L CNN
+F 0 "Q31" H 2575 5700 50  0000 L CNN
 F 1 "Q_NMOS_DGS" H 2575 5600 50  0000 L CNN
 F 2 "" H 2575 5750 50  0001 C CNN
@@
 Text Notes 4875 1175 0    157  ~ 0
 USB to UART\n
+NoConn ~ 7025 3225
+NoConn ~ 7025 3375
+NoConn ~ 7025 3450
+NoConn ~ 7025 3600
+NoConn ~ 7025 3675
+NoConn ~ 7025 3750
+NoConn ~ 7025 3825
+NoConn ~ 7025 3900
+NoConn ~ 7025 3975
+NoConn ~ 7025 4050
+NoConn ~ 7025 4125
+NoConn ~ 7025 4400
+NoConn ~ 7025 4475
+NoConn ~ 7025 4550
+NoConn ~ 7025 4625
+NoConn ~ 7025 4700
+NoConn ~ 7025 4775
+NoConn ~ 7025 4950
+NoConn ~ 7025 5025
+NoConn ~ 7025 5100
+NoConn ~ 7025 5175
+NoConn ~ 7025 5675
+NoConn ~ 7025 5600
+NoConn ~ 7025 5475
+NoConn ~ 7025 5400
+NoConn ~ 7025 5325
+NoConn ~ 7025 5250
 $EndSCHEMATC

Commit message: arduino time
Parts:
- C24, C25, C26, C27, C28, C29, C30, C31, C32, C33, C34, C35, C37, C38, C39, C40: footprint (none) -> Capacitors_SMD:C_0603
- D7, D8: footprint (none) -> project2:PBG1010603
- FB1, FB2: footprint (none) -> project2:240-2399-1-ND
- Q31: footprint (none) -> TO_SOT_Packages_SMD:SOT-363_SC-70-6
- R10, R12, R23, R24, R25, R26: footprint (none) -> Resistors_SMD:R_0603
- Y2: footprint (none) -> Crystals:Crystal_SMD_Abracon_ABM8G-4pin_3.2x2.5mm
Changed lines of the file:
@@
 F 0 "C40" H 5125 5600 50  0000 L CNN
 F 1 "12pF" H 5125 5400 50  0000 L CNN
-F 2 "" H 5138 5350 50  0001 C CNN
+F 2 "Capacitors_SMD:C_0603" H 5138 5350 50  0001 C CNN
 F 3 "" H 5100 5500 50  0001 C CNN
 	1    5100 5500
@@
 F 0 "C39" H 3875 5600 50  0000 L CNN
 F 1 "12pF" H 3875 5400 50  0000 L CNN
-F 2 "" H 3888 5350 50  0001 C CNN
+F 2 "Capacitors_SMD:C_0603" H 3888 5350 50  0001 C CNN
 F 3 "" H 3850 5500 50  0001 C CNN
 	1    3850 5500
@@
 F 0 "Y2" H 4525 5275 60  0000 C CNN
 F 1 "12Mhz" H 4525 5125 60  0000 C CNN
-F 2 "" H 4525 5100 60  0001 C CNN
+F 2 "Crystals:Crystal_SMD_Abracon_ABM8G-4pin_3.2x2.5mm" H 4525 5100 60  0001 C CNN
 F 3 "" H 4525 5100 60  0001 C CNN
 	1    4525 5100
@@
 F 0 "FB1" V 4375 1675 50  0000 C CNN
 F 1 "Ferrite_Bead" V 4675 1650 50  0000 C CNN
-F 2 "" V 4455 1650 50  0001 C CNN
+F 2 "project2:240-2399-1-ND" V 4455 1650 50  0001 C CNN
 F 3 "" H 4525 1650 50  0001 C CNN
 	1    4525 1650
@@
 F 0 "FB2" V 4375 2300 50  0000 C CNN
 F 1 "Ferrite_Bead" V 4675 2275 50  0000 C CNN
-F 2 "" V 4455 2275 50  0001 C CNN
+F 2 "project2:240-2399-1-ND" V 4455 2275 50  0001 C CNN
 F 3 "" H 4525 2275 50  0001 C CNN
 	1    4525 2275
@@
 F 0 "C24" H 5075 1900 50  0000 L CNN
 F 1 "4.7nF" H 5075 1700 50  0000 L CNN
-F 2 "" H 5088 1650 50  0001 C CNN
+F 2 "Capacitors_SMD:C_0603" H 5088 1650 50  0001 C CNN
 F 3 "" H 5050 1800 50  0001 C CNN
 	1    5050 1800
@@
 F 0 "C25" H 5450 1900 50  0000 L CNN
 F 1 ".1uF" H 5450 1700 50  0000 L CNN
-F 2 "" H 5463 1650 50  0001 C CNN
+F 2 "Capacitors_SMD:C_0603" H 5463 1650 50  0001 C CNN
 F 3 "" H 5425 1800 50  0001 C CNN
 	1    5425 1800
@@
 F 0 "C32" H 5075 2525 50  0000 L CNN
 F 1 "4.7nF" H 5075 2325 50  0000 L CNN
-F 2 "" H 5088 2275 50  0001 C CNN
+F 2 "Capacitors_SMD:C_0603" H 5088 2275 50  0001 C CNN
 F 3 "" H 5050 2425 50  0001 C CNN
 	1    5050 2425
@@
 F 0 "C33" H 5450 2525 50  0000 L CNN
 F 1 ".1uF" H 5450 2325 50  0000 L CNN
-F 2 "" H 5463 2275 50  0001 C CNN
+F 2 "Capacitors_SMD:C_0603" H 5463 2275 50  0001 C CNN
 F 3 "" H 5425 2425 50  0001 C CNN
 	1    5425 2425
@@
 F 0 "C34" H 4100 3625 50  0000 L CNN
 F 1 ".1uF" H 4100 3425 50  0000 L CNN
-F 2 "" H 4113 3375 50  0001 C CNN
+F 2 "Capacitors_SMD:C_0603" H 4113 3375 50  0001 C CNN
 F 3 "" H 4075 3525 50  0001 C CNN
 	1    4075 3525
@@
 F 0 "C37" H 4900 3600 50  0000 L CNN
 F 1 "4.7nF" H 4900 3400 50  0000 L CNN
-F 2 "" H 4913 3350 50  0001 C CNN
+F 2 "Capacitors_SMD:C_0603" H 4913 3350 50  0001 C CNN
 F 3 "" H 4875 3500 50  0001 C CNN
 	1    4875 3500
@@
 F 0 "C38" H 5200 3600 50  0000 L CNN
 F 1 ".1uF" H 5200 3400 50  0000 L CNN
-F 2 "" H 5213 3350 50  0001 C CNN
+F 2 "Capacitors_SMD:C_0603" H 5213 3350 50  0001 C CNN
 F 3 "" H 5175 3500 50  0001 C CNN
 	1    5175 3500
@@
 F 0 "C35" H 3325 3350 50  0000 L CNN
 F 1 "4.7uF" H 3325 3150 50  0000 L CNN
-F 2 "" H 3338 3100 50  0001 C CNN
+F 2 "Capacitors_SMD:C_0603" H 3338 3100 50  0001 C CNN
 F 3 "" H 3300 3250 50  0001 C CNN
 	1    3300 3250
@@
 F 0 "D7" H 3175 4675 60  0000 C CNN
 F 1 "PGB1010603" H 3225 4400 60  0000 C CNN
-F 2 "" H 3225 4575 60  0001 C CNN
+F 2 "project2:PBG1010603" H 3225 4575 60  0001 C CNN
 F 3 "" H 3225 4575 60  0001 C CNN
 	1    3225 4575
@@
 F 0 "D8" H 3600 4675 60  0000 C CNN
 F 1 "PGB1010603" H 3650 4400 60  0000 C CNN
-F 2 "" H 3650 4575 60  0001 C CNN
+F 2 "project2:PBG1010603" H 3650 4575 60  0001 C CNN
 F 3 "" H 3650 4575 60  0001 C CNN
 	1    3650 4575
@@
 F 0 "R24" V 5330 4525 50  0000 C CNN
 F 1 "12K" V 5250 4525 50  0000 C CNN
-F 2 "" V 5180 4525 50  0001 C CNN
+F 2 "Resistors_SMD:R_0603" V 5180 4525 50  0001 C CNN
 F 3 "" H 5250 4525 50  0001 C CNN
 	1    5250 4525
@@
 F 0 "R23" V 3005 5600 50  0000 C CNN
 F 1 "12K" V 2925 5600 50  0000 C CNN
-F 2 "" V 2855 5600 50  0001 C CNN
+F 2 "Resistors_SMD:R_0603" V 2855 5600 50  0001 C CNN
 F 3 "" H 2925 5600 50  0001 C CNN
 	1    2925 5600
@@
 F 0 "R10" V 7205 3500 50  0000 C CNN
 F 1 "1K" V 7125 3500 50  0000 C CNN
-F 2 "" V 7055 3500 50  0001 C CNN
+F 2 "Resistors_SMD:R_0603" V 7055 3500 50  0001 C CNN
 F 3 "" H 7125 3500 50  0001 C CNN
 	1    7125 3500
@@
 F 0 "R12" V 7380 3500 50  0000 C CNN
 F 1 "1K" V 7300 3500 50  0000 C CNN
-F 2 "" V 7230 3500 50  0001 C CNN
+F 2 "Resistors_SMD:R_0603" V 7230 3500 50  0001 C CNN
 F 3 "" H 7300 3500 50  0001 C CNN
 	1    7300 3500
@@
 F 0 "R25" V 7525 4275 50  0000 C CNN
 F 1 "1K" V 7625 4250 50  0000 C CNN
-F 2 "" V 7555 4250 50  0001 C CNN
+F 2 "Resistors_SMD:R_0603" V 7555 4250 50  0001 C CNN
 F 3 "" H 7625 4250 50  0001 C CNN
 	1    7625 4250
@@
 F 0 "R26" V 7355 4475 50  0000 C CNN
 F 1 "1K" V 7275 4475 50  0000 C CNN
-F 2 "" V 7205 4475 50  0001 C CNN
+F 2 "Resistors_SMD:R_0603" V 7205 4475 50  0001 C CNN
 F 3 "" H 7275 4475 50  0001 C CNN
 	1    7275 4475
@@
 F 0 "C26" H 6850 2375 50  0000 L CNN
 F 1 ".1uF" H 6850 2175 50  0000 L CNN
-F 2 "" H 6863 2125 50  0001 C CNN
+F 2 "Capacitors_SMD:C_0603" H 6863 2125 50  0001 C CNN
 F 3 "" H 6825 2275 50  0001 C CNN
 	1    6825 2275
@@
 F 0 "C27" H 7150 2375 50  0000 L CNN
 F 1 ".1uF" H 7150 2175 50  0000 L CNN
-F 2 "" H 7163 2125 50  0001 C CNN
+F 2 "Capacitors_SMD:C_0603" H 7163 2125 50  0001 C CNN
 F 3 "" H 7125 2275 50  0001 C CNN
 	1    7125 2275
@@
 F 0 "C28" H 7450 2375 50  0000 L CNN
 F 1 ".1uF" H 7450 2175 50  0000 L CNN
-F 2 "" H 7463 2125 50  0001 C CNN
+F 2 "Capacitors_SMD:C_0603" H 7463 2125 50  0001 C CNN
 F 3 "" H 7425 2275 50  0001 C CNN
 	1    7425 2275
@@
 F 0 "C29" H 8000 2350 50  0000 L CNN
 F 1 ".1uF" H 8000 2150 50  0000 L CNN
-F 2 "" H 8013 2100 50  0001 C CNN
+F 2 "Capacitors_SMD:C_0603" H 8013 2100 50  0001 C CNN
 F 3 "" H 7975 2250 50  0001 C CNN
 	1    7975 2250
@@
 F 0 "C30" H 8275 2350 50  0000 L CNN
 F 1 ".1uF" H 8275 2150 50  0000 L CNN
-F 2 "" H 8288 2100 50  0001 C CNN
+F 2 "Capacitors_SMD:C_0603" H 8288 2100 50  0001 C CNN
 F 3 "" H 8250 2250 50  0001 C CNN
 	1    8250 2250
@@
 F 0 "C31" H 8550 2350 50  0000 L CNN
 F 1 ".1uF" H 8550 2150 50  0000 L CNN
-F 2 "" H 8563 2100 50  0001 C CNN
+F 2 "Capacitors_SMD:C_0603" H 8563 2100 50  0001 C CNN
 F 3 "" H 8525 2250 50  0001 C CNN
 	1    8525 2250
@@
 F 0 "Q31" H 2575 5700 50  0000 L CNN
 F 1 "Q_NMOS_DGS" H 2575 5600 50  0000 L CNN
-F 2 "" H 2575 5750 50  0001 C CNN
+F 2 "TO_SOT_Packages_SMD:SOT-363_SC-70-6" H 2575 5750 50  0001 C CNN
 F 3 "" H 2375 5650 50  0001 C CNN
 	1    2375 5650
