File: Project 2_Arduino/Project 2_Arduino.sch (KiCad schematic (older format))
At the start: 4 parts, among them U3 ATMEGA328P-AU

Commit message: acheamic in progress
Parts:
- added C1: 100nF, symbol C
- added C3, C7: 1uF, symbol C
- added C5: 4.7uF_16V, symbol CP
- added C?: C, symbol C
- added D? (x2): D, symbol D
- added R? (x4): R, symbol R
- added U2: LM1117-5.0, symbol LM1117-5.0
Connections:
- net D11 is gone; now on net D11/MOSI: J?.4 (Pin_4)
- net D12 is gone; now on net D12/MISO: J?.5 (Pin_5)
- net D13 is gone; now on net D13/SCK: J?.6 (Pin_6)
- net D13/SCK: no longer U3.17 ((PCINT5/SCK)PB5)
- net GND: now also C1.2, C3.2, C5.2, C7.2, C?.2, D?.1 (K), U2.1 (GND)
- net 5V: now reaches U3.18 (AVCC)
- net 5V: now also U3.4 (VCC), U3.6 (VCC), C3.1, C5.1, C7.1, D?.1 (K)
- net at U3.20 (AREF): now also C1.1
- net D1/TX: now reaches U3.30 ((PCINT16/RXD)PD0)
- net D1/TX: now also R?.2
- net D0/RX: now reaches U3.31 ((PCINT17/TXD)PD1)
- net D0/RX: now also R?.2
- new net: C?.1, R?.2, U2.2 (VO)
- new net: R?.2, U3.17 ((PCINT5/SCK)PB5)
- new net: D?.2 (A), R?.1
- new net RX: R?.1
- new net TX: R?.1
- new net VIN: U2.3 (VI)
- new net VUSB: D?.2 (A)
